File: EC_RD/OGS_RD/Simulation/AFE_SIM_v1/AFE_SIM_v1.kicad_sch (KiCad schematic)
At the start: 81 parts, among them U1 ${SIM.PARAMS}, U2 ${SIM.PARAMS}, U3 ${SIM.PARAMS}, U4 ${SIM.PARAMS}, U5 ${SIM.PARAMS}, U6 ${SIM.PARAMS}, U7 ${SIM.PARAMS}

Commit message: update
Parts:
- I1: value 400n -> 0
- R17: value 1k -> 47k
Other:
- moved on the sheet: C4, C7
Changed lines of the file:
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@@
 	)
 	(junction
-		(at 113.03 52.705)
+		(at 175.26 41.91)
 		(diameter 0)
 		(color 0 0 0 0)
@@
 	)
 	(junction
-		(at 175.26 42.545)
-		(diameter 0)
-		(color 0 0 0 0)
-	)
-	(junction
 		(at 175.26 114.3)
 		(diameter 0)
@@
 	)
 	(junction
-		(at 52.07 116.205)
+		(at 113.03 53.34)
 		(diameter 0)
 		(color 0 0 0 0)
 	)
 	(junction
-		(at 175.26 60.325)
+		(at 52.07 116.205)
 		(diameter 0)
 		(color 0 0 0 0)
 	)
 	(junction
-		(at 113.03 42.545)
+		(at 175.26 60.325)
 		(diameter 0)
 		(color 0 0 0 0)
@@
 	)
 	(junction
+		(at 113.03 41.91)
+		(diameter 0)
+		(color 0 0 0 0)
+	)
+	(junction
 		(at 134.62 185.42)
 		(diameter 0)
@@
 	(wire
 		(pts
+			(xy 113.03 53.34) (xy 113.03 57.785)
+		)
+		(stroke
+			(width 0)
+			(type default)
+		)
+	)
+	(wire
+		(pts
 			(xy 175.26 157.48) (xy 175.26 167.64)
 		)
@@
 	(wire
 		(pts
+			(xy 127 41.91) (xy 134.62 41.91)
+		)
+		(stroke
+			(width 0)
+			(type default)
+		)
+	)
+	(wire
+		(pts
 			(xy 68.58 170.815) (xy 68.58 177.8)
 		)
@@
 	(wire
 		(pts
-			(xy 113.03 32.385) (xy 113.03 42.545)
+			(xy 140.97 49.53) (xy 140.97 32.385)
 		)
 		(stroke
@@
 	(wire
 		(pts
-			(xy 140.97 49.53) (xy 140.97 32.385)
+			(xy 113.03 41.91) (xy 113.03 53.34)
 		)
 		(stroke
@@
 	(wire
 		(pts
-			(xy 175.26 42.545) (xy 184.15 42.545)
-		)
-		(stroke
-			(width 0)
-			(type default)
-		)
-	)
-	(wire
-		(pts
 			(xy 175.26 60.325) (xy 175.26 62.865)
 		)
@@
 	(wire
 		(pts
-			(xy 97.79 50.165) (xy 97.79 52.705)
+			(xy 97.79 50.165) (xy 97.79 53.34)
 		)
 		(stroke
@@
 	(wire
 		(pts
-			(xy 175.26 42.545) (xy 175.26 55.245)
-		)
-		(stroke
-			(width 0)
-			(type default)
-		)
-	)
-	(wire
-		(pts
 			(xy 175.26 67.945) (xy 175.26 69.215)
 		)
@@
 	(wire
 		(pts
-			(xy 189.23 42.545) (xy 195.58 42.545)
-		)
-		(stroke
-			(width 0)
-			(type default)
-		)
-	)
-	(wire
-		(pts
 			(xy 210.82 182.88) (xy 204.47 182.88)
 		)
@@
 	(wire
 		(pts
-			(xy 134.62 60.325) (xy 134.62 42.545)
+			(xy 134.62 41.91) (xy 134.62 60.325)
 		)
 		(stroke
@@
 	(wire
 		(pts
+			(xy 97.79 53.34) (xy 113.03 53.34)
+		)
+		(stroke
+			(width 0)
+			(type default)
+		)
+	)
+	(wire
+		(pts
 			(xy 182.88 109.22) (xy 182.88 107.315)
 		)
@@
 	(wire
 		(pts
+			(xy 189.23 41.91) (xy 195.58 41.91)
+		)
+		(stroke
+			(width 0)
+			(type default)
+		)
+	)
+	(wire
+		(pts
 			(xy 97.79 177.8) (xy 113.03 177.8)
 		)
@@
 	(wire
 		(pts
-			(xy 113.03 42.545) (xy 121.92 42.545)
+			(xy 326.39 44.45) (xy 328.93 44.45)
 		)
 		(stroke
@@
 	(wire
 		(pts
-			(xy 326.39 44.45) (xy 328.93 44.45)
+			(xy 132.08 60.325) (xy 134.62 60.325)
 		)
 		(stroke
@@
 	(wire
 		(pts
-			(xy 132.08 60.325) (xy 134.62 60.325)
+			(xy 45.72 174.625) (xy 45.72 170.815)
 		)
 		(stroke
@@
 	(wire
 		(pts
-			(xy 45.72 174.625) (xy 45.72 170.815)
+			(xy 113.03 32.385) (xy 113.03 41.91)
 		)
 		(stroke
@@
 	(wire
 		(pts
-			(xy 113.03 52.705) (xy 113.03 57.785)
+			(xy 204.47 116.84) (xy 204.47 119.38)
 		)
 		(stroke
@@
 	(wire
 		(pts
-			(xy 204.47 116.84) (xy 204.47 119.38)
+			(xy 149.86 163.83) (xy 149.86 166.37)
 		)
 		(stroke
@@
 	(wire
 		(pts
-			(xy 149.86 163.83) (xy 149.86 166.37)
+			(xy 175.26 41.91) (xy 175.26 55.245)
 		)
 		(stroke
@@
 	(wire
 		(pts
-			(xy 97.79 52.705) (xy 113.03 52.705)
+			(xy 134.62 101.6) (xy 127 101.6)
 		)
 		(stroke
@@
 	(wire
 		(pts
-			(xy 134.62 101.6) (xy 127 101.6)
+			(xy 182.88 173.355) (xy 187.96 173.355)
 		)
 		(stroke
@@
 	(wire
 		(pts
-			(xy 182.88 173.355) (xy 187.96 173.355)
+			(xy 210.82 57.785) (xy 204.47 57.785)
 		)
 		(stroke
@@
 	(wire
 		(pts
-			(xy 210.82 57.785) (xy 204.47 57.785)
+			(xy 195.58 182.88) (xy 198.12 182.88)
 		)
 		(stroke
@@
 	(wire
 		(pts
-			(xy 195.58 182.88) (xy 198.12 182.88)
+			(xy 140.97 119.38) (xy 160.02 119.38)
 		)
 		(stroke
@@
 	(wire
 		(pts
-			(xy 140.97 119.38) (xy 160.02 119.38)
+			(xy 113.03 41.91) (xy 121.92 41.91)
 		)
 		(stroke
@@
 	(wire
 		(pts
-			(xy 113.03 42.545) (xy 113.03 52.705)
-		)
-		(stroke
-			(width 0)
-			(type default)
-		)
-	)
-	(wire
-		(pts
 			(xy 52.07 104.775) (xy 68.58 104.775)
 		)
@@
 	(wire
 		(pts
-			(xy 134.62 42.545) (xy 127 42.545)
-		)
-		(stroke
-			(width 0)
-			(type default)
-		)
-	)
-	(wire
-		(pts
 			(xy 149.86 100.33) (xy 149.86 101.6)
 		)
@@
 	(wire
 		(pts
-			(xy 175.26 32.385) (xy 175.26 42.545)
+			(xy 175.26 32.385) (xy 175.26 41.91)
 		)
 		(stroke
@@
 	(wire
 		(pts
-			(xy 195.58 42.545) (xy 195.58 57.785)
+			(xy 195.58 41.91) (xy 195.58 57.785)
 		)
 		(stroke
@@
 	(wire
 		(pts
+			(xy 175.26 41.91) (xy 184.15 41.91)
+		)
+		(stroke
+			(width 0)
+			(type default)
+		)
+	)
+	(wire
+		(pts
 			(xy 45.72 179.705) (xy 45.72 189.865)
 		)
@@
 	(symbol
 		(lib_id "Device:C_Small")
-		(at 186.69 42.545 270)
+		(at 186.69 41.91 270)
 		(unit 1)
 		(exclude_from_sim no)
@@
 		(dnp no)
 		(property "Reference" "C4"
-			(at 186.055 45.085 90)
+			(at 186.055 44.45 90)
 			(effects
 				(font
@@
 		)
 		(property "Value" "10nF"
-			(at 184.15 39.624 90)
+			(at 184.15 38.989 90)
 			(effects
 				(font
@@
 		)
 		(property "Footprint" "Capacitor_SMD:C_0603_1608Metric"
-			(at 186.69 42.545 0)
+			(at 186.69 41.91 0)
 			(effects
 				(font
@@
 		)
 		(property "Datasheet" "~"
-			(at 186.69 42.545 0)
+			(at 186.69 41.91 0)
 			(effects
 				(font
@@
 		)
 		(property "Description" ""
-			(at 186.69 42.545 0)
+			(at 186.69 41.91 0)
 			(effects
 				(font
@@
 			)
 		)
-		(property "Value" "400n"
+		(property "Value" "0"
 			(at 101.6 67.9449 0)
 			(effects
@@
 	(symbol
 		(lib_id "Device:C_Small")
-		(at 124.46 42.545 90)
+		(at 124.46 41.91 90)
 		(unit 1)
 		(exclude_from_sim no)
@@
 		(dnp no)
 		(property "Reference" "C7"
-			(at 125.095 40.005 90)
+			(at 125.095 39.37 90)
 			(effects
 				(font
@@
 		)
 		(property "Value" "220nF"
-			(at 126.365 45.085 90)
+			(at 126.365 44.45 90)
 			(effects
 				(font
@@
 		)
 		(property "Footprint" "Capacitor_SMD:C_0603_1608Metric"
-			(at 124.46 42.545 0)
+			(at 124.46 41.91 0)
 			(effects
 				(font
@@
 		)
 		(property "Datasheet" "~"
-			(at 124.46 42.545 0)
+			(at 124.46 41.91 0)
 			(effects
 				(font
@@
 		)
 		(property "Description" ""
-			(at 124.46 42.545 0)
+			(at 124.46 41.91 0)
 			(effects
 				(font
@@
 			)
 		)
-		(property "Value" "1k"
+		(property "Value" "47k"
 			(at 140.97 52.07 90)
 			(effects
