File: OZ_AFE_1/OZ_AFE_1.kicad_pcb (KiCad board)
At the start: 2 copper layers, 32 x 31 mm, 55 parts, among them U1 LT6011, U2 TLV2211, U3 ISL21009BFB825Z, U4 LT6011, U5 OGS, U6 MCP9700x-HTT

Commit message: New Simulation and PCB
Parts:
- removed R17, R18: 47K, Resistor_SMD:R_0603_1608Metric
- removed U3: ISL21009BFB825Z, Package_SO:SOIC-8_3.9x4.9mm_P1.27mm
- added U7: REF35250QDBVR, Package_TO_SOT_SMD:SOT-23-6, F.Cu at (119.5, 94.5)
- R12, R6: value 100K -> 147K
Connections:
- C5 pad 2: +6V -> +5V
- D1 pad 1: +6V -> +5V
- R12 pad 2: Net-(R12-Pad2) -> Net-(C7-Pad2)
- R16 pad 2: +6V -> +5V
- R6 pad 2: Net-(R18-Pad2) -> Net-(C1-Pad2)
- U1 pad 3: +2.5V -> VMID
- U4 pad 5: +2.5V -> VMID
- U5 pad 8: GNDA -> GND

Commit message: update
Parts:
- moved U1 52.5 mm to (162.0, 90.5)
- moved R11 28.1 mm to (140.8, 83.8), turned to 90 degrees
- moved U4 20.4 mm to (137.0, 86.0), turned to -90 degrees
- moved R14 18.9 mm to (139.0, 80.5), turned to -90 degrees
- moved C6 17.8 mm to (140.8, 80.5), turned to 90 degrees
- moved R13 12.9 mm to (137.2, 80.5), turned to 90 degrees
Connections:
- C2 pad 1: +6V -> +5V
- C8 pad 1: +6V -> +5V
- U1 pad 8: +6V -> +5V
- U4 pad 8: +6V -> +5V

Commit message: sch update
Parts:
- removed D1: BZV55-C6V8, Diode_SMD:D_MiniMELF
- removed U2: TLV2211, Package_TO_SOT_SMD:SOT-23-5
- added C14: 100nF, Capacitor_SMD:C_0603_1608Metric, F.Cu at (124.8, 81.8)
- added C15: 1uF, Capacitor_SMD:C_0603_1608Metric, F.Cu at (114.2, 75.5)
- added C16: 1nF, Capacitor_SMD:C_0402_1005Metric, F.Cu at (100.2, 88.0)
- added C17: 1nF, Capacitor_SMD:C_0402_1005Metric, F.Cu at (123.0, 88.2)
- added C18: 1nF, Capacitor_SMD:C_0402_1005Metric, F.Cu at (122.2, 73.0)
- added C19: 1nF, Capacitor_SMD:C_0402_1005Metric, F.Cu at (125.5, 90.5)
- added FB1: BLM21PG121SN1, Resistor_SMD:R_0805_2012Metric, F.Cu at (114.5, 72.2)
- added FB2: BLM21PG121SN1, Resistor_SMD:R_0805_2012Metric, F.Cu at (116.2, 75.5)
- added FB3: LQW18ANR47J00D, Inductor_SMD:L_0603_1608Metric, F.Cu at (125.5, 88.2)
- added FB4: LQW18ANR47J00D, Inductor_SMD:L_0603_1608Metric, F.Cu at (100.2, 85.2)
- added FB5: LQW18ANR47J00D, Inductor_SMD:L_0603_1608Metric, F.Cu at (122.8, 90.5)
- added FB6: LQW18ANR47J00D, Inductor_SMD:L_0603_1608Metric, F.Cu at (119.5, 74.8)
- added JP1: SolderJumper_3_Open, Jumper:SolderJumper-3_P1.3mm_Open_RoundedPad1.0x1.5mm, F.Cu at (128.8, 68.5)
- added JP2: SolderJumper_3_Open, Jumper:SolderJumper-3_P1.3mm_Open_RoundedPad1.0x1.5mm, F.Cu at (133.5, 68.5)
- added Q1: MMBFJ270, Package_TO_SOT_SMD:SOT-23, F.Cu at (125.5, 85.5)
- added Q2: MMBFJ270, Package_TO_SOT_SMD:SOT-23, F.Cu at (101.0, 80.2)
- added R17: 1M, Resistor_SMD:R_0402_1005Metric, F.Cu at (104.0, 80.2)
- added R5: 1M, Resistor_SMD:R_0402_1005Metric, F.Cu at (127.5, 82.8)
- added U3: TLV8811, Package_TO_SOT_SMD:SOT-23-6, F.Cu at (124.8, 78.8)
- C2: value 10uF -> 100nF
- R1, R10, R13, R14, R15, R2, R22, R23, R24, R25, R26, R27, R28, R3, R4, R9: footprint Resistor_SMD:R_0603_1608Metric -> Resistor_SMD:R_0402_1005Metric
- U1, U4: value LT6011 -> LT6011IMS8#PBF; footprint Package_SO:SOIC-8_3.9x4.9mm_P1.27mm -> Package_SO:MSOP-8_3x3mm_P0.65mm
- moved U1 53.8 mm to (108.5, 84.5)
- moved R1 22.3 mm to (115.8, 94.0), turned to 0 degrees
- moved R6B0 21.9 mm to (119.2, 92.2)
- moved C10 21.6 mm to (99.2, 60.2)
- moved U6 21.5 mm to (99.2, 63.2)
- moved C3 21.3 mm to (115.8, 92.2), turned to 180 degrees
- moved U4 21.3 mm to (115.8, 84.5), turned to 90 degrees
- moved C5 21.0 mm to (118.0, 72.2), turned to 180 degrees
- moved C11 20.9 mm to (108.5, 94.0), turned to 180 degrees
- moved U7 20.6 mm to (111.5, 75.5), turned to 90 degrees
- moved C13 20.5 mm to (107.5, 73.2), turned to -90 degrees
- moved R21 20.3 mm to (104.8, 73.2), turned to -90 degrees
- moved R25 18.5 mm to (118.5, 81.0), turned to -90 degrees
- moved R16 18.2 mm to (119.2, 70.0), turned to 0 degrees
- moved R29 17.5 mm to (122.8, 92.2), turned to 180 degrees
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Connections:
- C1 pad 1: Net-(U1A--) -> Net-(U1B--)
- C4 pad 2: Net-(U2--) -> Net-(U4A--)
- C9 pad 2: Net-(U1B--) -> Net-(U1A--)
- R11 pad 1: Net-(SN1-CE) -> Net-(C19-Pad2)
- R13 pad 1: Net-(SN1-RE) -> Net-(C18-Pad1)
- R14 pad 2: Net-(U4A--) -> Net-(U3--)
- R15 pad 1: Net-(SN1-WE) -> Net-(C17-Pad1)
- R19B0 pad 1: Net-(U1B--) -> Net-(U1A--)
- R2 pad 1: Net-(U1A--) -> Net-(U1B--)
- R2 pad 2: Net-(SN1-AE) -> Net-(C16-Pad1)
- R21B0 pad 1: Net-(U1B-+) -> Net-(U1A-+)
- R22 pad 1: Net-(U1B--) -> Net-(U1A--)
- R23 pad 1: Net-(U1B-+) -> Net-(U1A-+)
- R26 pad 2: Net-(U1A--) -> Net-(U1B--)
- R4 pad 1: Net-(U2--) -> Net-(U4A--)
- R6 pad 1: Net-(U1A--) -> Net-(U1B--)
- R6B0 pad 1: Net-(U2--) -> Net-(U4A--)
- R7B0 pad 1: Net-(U2-+) -> Net-(U4A-+)
- R9 pad 1: Net-(U2-+) -> Net-(U4A-+)
- SN1 pad 1: Net-(SN1-AE) -> AUX
- SN1 pad 2: Net-(SN1-RE) -> REF
- SN1 pad 3: Net-(SN1-WE) -> WORK
- U1 pad 1: Net-(C1-Pad2) -> Net-(C9-Pad1)
- U1 pad 3: VMID -> Net-(U1A-+)
- U1 pad 5: Net-(U1B-+) -> VMID
- U1 pad 7: Net-(C9-Pad1) -> Net-(C1-Pad2)
- U4 pad 1: Net-(C6-Pad1) -> Net-(C4-Pad1)
- U4 pad 3: +2.5V -> Net-(U4A-+)
